File: FirstArdTest/Something/Something.kicad_sch (KiCad schematic)
At the start: 16 parts, among them J1 USBC Connector, Q1 NMOS, Q2 NMOS, U1 BatIC-MCP73831, U2 BattSafety

Commit message: PD realization commit
Parts:
- removed C1: 4.7uF, symbol Device:C
- added A?: Arduino_Nano_v3.x, Module:Arduino_Nano, symbol MCU_Module:Arduino_Nano_v3.x
- added C4, C?, CVB2, CVB?: 22uF, symbol Device:C
- added CVB1, CVB?: 0.1uF, symbol Device:C
- added CVB? (x2): 1uF, symbol Device:C
- added D? (x2): ESD441DPLR, ESD441DPLR, symbol SamacSys_Parts:ESD441DPLR
- added D? (x2): ESD321DPYR, DPY(R-PX1SON-N2), symbol SamacSys_Parts:ESD321DPYR
- added D?: SS34, Diode_SMD:D_SMA, symbol Diode:SS34
- added IC?: STUSB4531BJR, BGA16C40P4X4_226X226X54, symbol SamacSys_Parts:STUSB4531BJR
- added L1: 4.7uH, symbol Device:L
- added U?: MT3608, Package_TO_SOT_SMD:SOT-23-6, symbol Regulator_Switching:MT3608
- R5: value 5.1k -> 110k
- R6: value 5.1k -> 15k
- renumbered U2 to DW01A
Connections:
- net P- is gone; now on net GND: Q2.1 (S1), Q2.3 (S2), R4.1
- net GND: now also C3.2, DW01A.6 (GND), LI-IONbatt.2, Q1.1 (S1), Q1.3 (S2), R2.2, R6.1, U1.2 (V_{SS}), A?.29 (GND), A?.4 (GND), C4.2, C?.2, CVB1.2, CVB2.2, CVB?.2, CVB?.2, CVB?.2, CVB?.2, U?.2 (GND)
- net P+: now also C4.1, L1.1, U?.4 (EN), U?.5 (IN)
- net V in: now also D?.2 (A); no longer D1.2 (A), U1.4 (V_{DD})
- net at J1.A1 (GND), J1.A12 (GND__1), J1.B1 (GND__2)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: now also D?.2 (A); no longer R2.2, R5.2, R6.2, U1.2 (V_{SS})
- net at J1.A5 (CC1): now also D?.1; no longer R6.1
- net at J1.B5 (CC2): now also D?.1; no longer R5.1
- new net: CVB1.1, CVB2.1, D?.1 (K), IC?.A1 (VDD)
- new net: D?.2, IC?.A2 (CC1)
- new net: D?.2, IC?.A3 (CC2)
- new net: CVB?.1, IC?.B1 (VREG_2V7)
- new net: CVB?.1, IC?.C1 (VREG_1V2)
- new net: CVB?.1, CVB?.1, D?.1 (K), IC?.D2 (GND)
- new net: R5.1, R6.2, U?.3 (FB)
- new net: D?.2 (A), L1.2, U?.1 (SW)
- new net: D1.2 (A), U1.4 (V_{DD})
- new net 5V out: A?.27 (+5V), C?.1, D?.1 (K), R5.2
Other:
- added sheet Pt2 (something2.kicad_sch)
- moved on the sheet: C2, C3, D1, DW01A, J1, LI-IONbatt, Q1, Q2, R1, R2, R3, R4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

Commit message: Almost done schematic push
Parts:
- added C?: 0.1uF, symbol Device:C
- CVB2, CVB?: value 22uF -> 10uF
Connections:
- net 5V out: now also C?.1; no longer A?.27 (+5V)
- net GND: now also D?.1 (K), D?.1 (K), D?.2, D?.2, C?.2
- net V in: now also CVB1.1, CVB2.1, IC?.A1 (VDD)
- net at IC?.A2 (CC1): now also D?.1, J1.A5 (CC1); no longer D?.2
- net at IC?.A3 (CC2): now also D?.1, J1.B5 (CC2); no longer D?.2
- net at CVB?.1, CVB?.1, IC?.D2 (GND): now also D?.2 (A), J1.A1 (GND), J1.A12 (GND__1), J1.B1 (GND__2), J1.B12 (GND__3); no longer D?.1 (K)
Other:
- moved on the sheet: CVB1, CVB2, D?
