File: FirstArdTest/Just theOLED/minithing/minithing.kicad_sch (KiCad schematic)
At the start: 35 parts, among them Q1 NMOS, Q2 NMOS, Q3 FDN340P, U1 TP4056-42-ESOP8, U2 MT3608

Commit message: Tahoe trip push
Parts:
- added SW? (x4): SW_Push, symbol Switch:SW_Push
- added U?: MCP23008-xSO, Package_SO:SOIC-18W_7.5x11.6mm_P1.27mm, symbol Interface_Expansion:MCP23008-xSO
Connections:
- net GND: now also U?.5 (GND), SW?.2, SW?.2, SW?.2, SW?.2, U?.3 (A2), U?.4 (A1), U?.5 (A0), U?.9 (VSS)
- net at C1.1, C2.1, C4.1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: no longer IC?.2 (VCC)
- net at IC?.7 (SDA): now also A1.24 (A5), U?.4 (SDA), U?.2 (SDA); no longer A1.23 (A4)
- net at IC?.8 (SCL): now also A1.23 (A4), U?.3 (SCL), U?.1 (SCL); no longer A1.24 (A5)
- net at U?.2 (VDD): now also A1.17 (3V3), IC?.2 (VCC), U?.18 (VDD)
- new net: SW?.1, U?.10 (GP0)
- new net: SW?.1, U?.11 (GP1)
- new net: SW?.1, U?.13 (GP3)
- new net: SW?.1, U?.12 (GP2)
Other:
- note added: "6/17/2026"
- moved on the sheet: A1, C5, IC?, R10, R7, R8, U1, U?
