File: FirstArdTest/Just theOLED/minithing/minithing.kicad_sch (KiCad schematic)
At the start: 40 parts, among them Q1 NMOS, Q2 NMOS, Q3 FDN340P, U1 TP4056-42-ESOP8, U2 MT3608

Commit message: PCB Finish
Parts:
- removed D1: ESD441DPLR, ESD441DPLR, symbol SamacSys_Parts:ESD441DPLR
- added Z1: 1N4733A, SamacSys_Parts:DIOAD1405W86L465D235, symbol SamacSys_Parts:1N4733A
- C1, C4, C7: footprint (none) -> Capacitor_SMD:C_1206_3216Metric_Pad1.33x1.80mm_HandSolder
- C2, C3, C5, C6, C8: footprint (none) -> Capacitor_SMD:C_0805_2012Metric_Pad1.18x1.45mm_HandSolder
- D2, D3: footprint Diode_SMD:D_SMA -> Diode_SMD:D_SMC_Handsoldering
- IC1: renamed from IC?; footprint SOIC127P600X175-8N -> SamacSys_Parts:SOIC127P600X175-8N
- J1: renamed from J?; footprint USB4110GFA -> SamacSys_Parts:USB4110GFA
- L1: footprint (none) -> Inductor_SMD:L_0805_2012Metric_Pad1.15x1.40mm_HandSolder
- LI-IONbatt1: footprint (none) -> Battery:BatteryHolder_Keystone_1042_1x18650
- Q1, Q2: footprint SOT95P280X125-6N -> SamacSys_Parts:SOT95P280X125-6N
- R1, R10, R11, R12, R2, R3, R4, R5, R6, R7, R8: footprint (none) -> Resistor_SMD:R_0805_2012Metric_Pad1.20x1.40mm_HandSolder
- R9: footprint (none) -> Resistor_SMD:R_1206_3216Metric_Pad1.30x1.75mm_HandSolder
- SW1, SW2, SW3, SW4: renamed from SW?; footprint (none) -> Button_Switch_THT:SW_PUSH_6mm
- U3: renamed from U?; footprint AHT20 -> SamacSys_Parts:AHT20
- gave numbers to parts that had none: 1
Connections:
- net GND: now also C3.2, DW01A1.6 (GND), LI-IONbatt1.2, Q1.1 (S1), Q1.3 (S2), Z1.1; no longer A1.6 (D3), R8.2, U1.7 (~{CHRG})
- net BATTERY: now reaches C5.1, LI-IONbatt1.1, Q3.2 (S), R11.2, R3.2, U1.5 (BAT)
- net 1AMP: now reaches C1.1, C2.1, C4.1, D2.2 (A2), J1.A4, J1.A9, J1.B4, J1.B9, L1.1, Q3.1 (G), Q3.3 (D), R9.1, U2.4 (EN), U2.5 (IN)
- net 1AMP: now also Z1.2
- new net: A1.6 (D3), R8.2, U1.7 (~{CHRG})

Commit message: Actual finish arduino pin change
Connections:
- net at C6.2, R11.1, R12.1: now also A1.19 (A0); no longer A1.7 (D4)

Commit message: Routine PCB ordered push, partial code
Parts:
- removed Z1: 1N4733A, SamacSys_Parts:DIOAD1405W86L465D235, symbol SamacSys_Parts:1N4733A
- D2: footprint Diode_SMD:D_SMC_Handsoldering -> Diode_SMD:D_SMA
Connections:
- net 5V out is gone; now on net 1AMP: A1.27 (+5V), C7.1, C8.2, D3.1 (K), R5.2
- net 1AMP: now also D2.1 (A1); no longer C4.1, D2.2 (A2), L1.1, Q3.3 (D), U2.4 (EN), U2.5 (IN)
- net GND: now also D2.2 (A2); no longer D2.1 (A1)
- new net: C4.1, L1.1, Q3.3 (D), U2.4 (EN), U2.5 (IN)
Other:
- moved on the sheet: D2

Commit message: LastFinalFinalPush
Parts:
- added R? (x2): 5.1KR, Resistor_SMD:R_0805_2012Metric_Pad1.20x1.40mm_HandSolder, symbol Device:R
Connections:
- net at A1.17 (3V3), IC1.2 (VCC), U3.2 (VDD)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: now also R?.1, R?.1
- net at A1.24 (A5), IC1.7 (SDA), U3.4 (SDA)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: now also R?.2
- net at A1.23 (A4), IC1.8 (SCL), U3.3 (SCL)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: now also R?.2
Changed lines of the file:
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@@
 	)
 	(junction
+		(at 265.43 120.65)
+		(diameter 0)
+		(color 0 0 0 0)
+	)
+	(junction
 		(at 242.57 71.12)
 		(diameter 0)
@@
 	)
 	(junction
+		(at 259.08 90.17)
+		(diameter 0)
+		(color 0 0 0 0)
+	)
+	(junction
 		(at 193.04 95.25)
 		(diameter 0)
@@
 	)
 	(junction
+		(at 259.08 118.11)
+		(diameter 0)
+		(color 0 0 0 0)
+	)
+	(junction
 		(at 179.07 135.89)
 		(diameter 0)
@@
 	)
 	(junction
+		(at 247.65 90.17)
+		(diameter 0)
+		(color 0 0 0 0)
+	)
+	(junction
 		(at 278.13 133.35)
 		(diameter 0)
@@
 	(wire
 		(pts
+			(xy 259.08 102.87) (xy 259.08 118.11)
+		)
+		(stroke
+			(width 0)
+			(type default)
+		)
+	)
+	(wire
+		(pts
 			(xy 236.22 156.21) (xy 242.57 156.21)
 		)
@@
 	(wire
 		(pts
+			(xy 259.08 118.11) (xy 278.13 118.11)
+		)
+		(stroke
+			(width 0)
+			(type default)
+		)
+	)
+	(wire
+		(pts
 			(xy 48.26 81.28) (xy 44.45 81.28)
 		)
@@
 	(wire
 		(pts
+			(xy 265.43 90.17) (xy 265.43 95.25)
+		)
+		(stroke
+			(width 0)
+			(type default)
+		)
+	)
+	(wire
+		(pts
 			(xy 182.88 113.03) (xy 182.88 139.7)
 		)
@@
 	(wire
 		(pts
+			(xy 247.65 90.17) (xy 247.65 129.54)
+		)
+		(stroke
+			(width 0)
+			(type default)
+		)
+	)
+	(wire
+		(pts
 			(xy 110.49 82.55) (xy 110.49 83.82)
 		)
@@
 	(wire
 		(pts
-			(xy 245.11 118.11) (xy 278.13 118.11)
+			(xy 245.11 118.11) (xy 259.08 118.11)
+		)
+		(stroke
+			(width 0)
+			(type default)
+		)
+	)
+	(wire
+		(pts
+			(xy 259.08 90.17) (xy 259.08 95.25)
 		)
 		(stroke
@@
 	(wire
 		(pts
+			(xy 265.43 102.87) (xy 265.43 120.65)
+		)
+		(stroke
+			(width 0)
+			(type default)
+		)
+	)
+	(wire
+		(pts
 			(xy 275.59 135.89) (xy 275.59 158.75)
 		)
@@
 	(wire
 		(pts
+			(xy 265.43 120.65) (xy 275.59 120.65)
+		)
+		(stroke
+			(width 0)
+			(type default)
+		)
+	)
+	(wire
+		(pts
 			(xy 191.77 58.42) (xy 191.77 60.96)
 		)
@@
 	(wire
 		(pts
+			(xy 259.08 90.17) (xy 265.43 90.17)
+		)
+		(stroke
+			(width 0)
+			(type default)
+		)
+	)
+	(wire
+		(pts
 			(xy 140.97 121.92) (xy 138.43 121.92)
 		)
@@
 	(wire
 		(pts
-			(xy 248.92 120.65) (xy 275.59 120.65)
+			(xy 248.92 120.65) (xy 265.43 120.65)
 		)
 		(stroke
@@
 	(wire
 		(pts
+			(xy 247.65 90.17) (xy 259.08 90.17)
+		)
+		(stroke
+			(width 0)
+			(type default)
+		)
+	)
+	(wire
+		(pts
 			(xy 189.23 148.59) (xy 189.23 115.57)
 		)
@@
 	(wire
 		(pts
-			(xy 247.65 82.55) (xy 247.65 129.54)
+			(xy 247.65 82.55) (xy 247.65 90.17)
 		)
 		(stroke
@@
 	)
 	(symbol
+		(lib_id "Device:R")
+		(at 265.43 99.06 0)
+		(mirror y)
+		(unit 1)
+		(exclude_from_sim no)
+		(in_bom yes)
+		(on_board yes)
+		(dnp no)
+		(property "Reference" "R?"
+			(at 270.256 97.536 0)
+			(effects
+				(font
+					(size 1.27 1.27)
+				)
+				(justify left)
+			)
+		)
+		(property "Value" "5.1KR"
+			(at 270.256 100.076 0)
+			(effects
+				(font
+					(size 1.27 1.27)
+				)
+				(justify left)
+			)
+		)
+		(property "Footprint" "Resistor_SMD:R_0805_2012Metric_Pad1.20x1.40mm_HandSolder"
+			(at 267.208 99.06 90)
+			(effects
+				(font
+					(size 1.27 1.27)
+				)
+				(hide yes)
+			)
+		)
+		(property "Datasheet" "~"
+			(at 265.43 99.06 0)
+			(effects
+				(font
+					(size 1.27 1.27)
+				)
+				(hide yes)
+			)
+		)
+		(property "Description" "Resistor"
+			(at 265.43 99.06 0)
+			(effects
+				(font
+					(size 1.27 1.27)
+				)
+				(hide yes)
+			)
+		)
+		(pin "1"
+		)
+		(pin "2"
+		)
+		(instances
+			(project "minithing"
+				(path "/d717513f-228d-40ff-a576-44c7a34457d9"
+					(reference "R?")
+					(unit 1)
+				)
+			)
+		)
+	)
+	(symbol
 		(lib_id "power:GND")
 		(at 278.13 53.34 90)
@@
 					(unit 1)
 				)
+			)
+		)
+	)
+	(symbol
+		(lib_id "Device:R")
+		(at 259.08 99.06 0)
+		(unit 1)
+		(exclude_from_sim no)
+		(in_bom yes)
+		(on_board yes)
+		(dnp no)
+		(property "Reference" "R?"
+			(at 254.254 97.536 0)
+			(effects
+				(font
+					(size 1.27 1.27)
+				)
+				(justify left)
+			)
+		)
+		(property "Value" "5.1KR"
+			(at 254.254 100.076 0)
+			(effects
+				(font
+					(size 1.27 1.27)
+				)
+				(justify left)
+			)
+		)
+		(property "Footprint" "Resistor_SMD:R_0805_2012Metric_Pad1.20x1.40mm_HandSolder"
+			(at 257.302 99.06 90)
+			(effects
+				(font
+					(size 1.27 1.27)
+				)
+				(hide yes)
+			)
+		)
+		(property "Datasheet" "~"
+			(at 259.08 99.06 0)
+			(effects
+				(font
+					(size 1.27 1.27)
+				)
+				(hide yes)
+			)
+		)
+		(property "Description" "Resistor"
+			(at 259.08 99.06 0)
+			(effects
+				(font
+					(size 1.27 1.27)
+				)
+				(hide yes)
+			)
+		)
+		(pin "1"
+		)
+		(pin "2"
+		)
+		(instances
+			(project "minithing"
+				(path "/d717513f-228d-40ff-a576-44c7a34457d9"
+					(reference "R?")
+					(unit 1)
+				)

Commit message: DEADASS final finish last frealsies
Parts:
- gave numbers to parts that had none: 2
Connections:
- net at IC1.7 (SDA), R14.2, U3.4 (SDA)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: now also A1.23 (A4); no longer A1.24 (A5)
- net at IC1.8 (SCL), R13.2, U3.3 (SCL)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: now also A1.24 (A5); no longer A1.23 (A4)
Changed lines of the file:
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@@
 	)
 	(junction
-		(at 245.11 118.11)
-		(diameter 0)
-		(color 0 0 0 0)
-	)
-	(junction
 		(at 191.77 60.96)
 		(diameter 0)
@@
 	)
 	(junction
+		(at 245.11 118.11)
+		(diameter 0)
+		(color 0 0 0 0)
+	)
+	(junction
 		(at 139.7 144.78)
 		(diameter 0)
@@
 	)
 	(junction
-		(at 248.92 120.65)
-		(diameter 0)
-		(color 0 0 0 0)
-	)
-	(junction
 		(at 275.59 135.89)
 		(diameter 0)
@@
 	)
 	(junction
+		(at 248.92 119.38)
+		(diameter 0)
+		(color 0 0 0 0)
+	)
+	(junction
 		(at 278.13 133.35)
 		(diameter 0)
@@
 	(wire
 		(pts
-			(xy 248.92 120.65) (xy 248.92 77.47)
+			(xy 248.92 120.65) (xy 248.92 119.38)
 		)
 		(stroke
@@
 	(wire
 		(pts
-			(xy 245.11 119.38) (xy 245.11 118.11)
-		)
-		(stroke
-			(width 0)
-			(type default)
-		)
-	)
-	(wire
-		(pts
 			(xy 242.57 158.75) (xy 242.57 162.56)
 		)
@@
 	(wire
 		(pts
+			(xy 248.92 119.38) (xy 248.92 77.47)
+		)
+		(stroke
+			(width 0)
+			(type default)
+		)
+	)
+	(wire
+		(pts
 			(xy 48.26 81.28) (xy 44.45 81.28)
 		)
@@
 	(wire
 		(pts
-			(xy 242.57 121.92) (xy 248.92 121.92)
-		)
-		(stroke
-			(width 0)
-			(type default)
-		)
-	)
-	(wire
-		(pts
-			(xy 248.92 121.92) (xy 248.92 120.65)
+			(xy 242.57 121.92) (xy 245.11 121.92)
 		)
 		(stroke
@@
 	(wire
 		(pts
+			(xy 242.57 119.38) (xy 248.92 119.38)
+		)
+		(stroke
+			(width 0)
+			(type default)
+		)
+	)
+	(wire
+		(pts
 			(xy 46.99 83.82) (xy 44.45 83.82)
 		)
@@
 	(wire
 		(pts
-			(xy 176.53 45.72) (xy 234.95 45.72)
+			(xy 245.11 118.11) (xy 245.11 121.92)
 		)
 		(stroke
@@
 	(wire
 		(pts
-			(xy 242.57 119.38) (xy 245.11 119.38)
+			(xy 176.53 45.72) (xy 234.95 45.72)
 		)
 		(stroke
@@
 		(on_board yes)
 		(dnp no)
-		(property "Reference" "R?"
+		(property "Reference" "R14"
 			(at 270.256 97.536 0)
 			(effects
@@
 			(project "minithing"
 				(path "/d717513f-228d-40ff-a576-44c7a34457d9"
-					(reference "R?")
+					(reference "R14")
 					(unit 1)
 				)
@@
 		(on_board yes)
 		(dnp no)
-		(property "Reference" "R?"
+		(property "Reference" "R13"
 			(at 254.254 97.536 0)
 			(effects
@@
 			(project "minithing"
 				(path "/d717513f-228d-40ff-a576-44c7a34457d9"
-					(reference "R?")
+					(reference "R13")
 					(unit 1)
 				)

Commit message: Picture input push
Connections:
- net BATTERY: now also Q3.3 (D); no longer Q3.2 (S)
- net at C4.1, L1.1, U2.4 (EN)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: now also Q3.2 (S); no longer Q3.3 (D)
Changed lines of the file:
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@@
+	)
+	(junction
+		(at 19.05 71.12)
+		(diameter 0)
+		(color 0 0 0 0)
+	)
+	(junction
+		(at 154.94 109.22)
+		(diameter 0)
+		(color 0 0 0 0)
+	)
+	(junction
+		(at 15.24 88.9)
+		(diameter 0)
+		(color 0 0 0 0)
+	)
+	(junction
+		(at 245.11 118.11)
+		(diameter 0)
+		(color 0 0 0 0)
+	)
+	(junction
+		(at 139.7 144.78)
+		(diameter 0)
+		(color 0 0 0 0)
+	)
+	(junction
+		(at 196.85 95.25)
+		(diameter 0)
+		(color 0 0 0 0)
+	)
+	(junction
+		(at 148.59 82.55)
+		(diameter 0)
+		(color 0 0 0 0)
+	)
+	(junction
+		(at 151.13 109.22)
+		(diameter 0)
+		(color 0 0 0 0)
+	)
+	(junction
+		(at 189.23 115.57)
+		(diameter 0)
+		(color 0 0 0 0)
+	)
+	(junction
+		(at 232.41 82.55)
+		(diameter 0)
+		(color 0 0 0 0)
+	)
+	(junction
+		(at 154.94 92.71)
+		(diameter 0)
+		(color 0 0 0 0)
+	)
+	(junction
+		(at 110.49 83.82)
+		(diameter 0)
+		(color 0 0 0 0)
+	)
+	(junction
+		(at 152.4 53.34)
+		(diameter 0)
+		(color 0 0 0 0)
+	)
+	(junction
+		(at 181.61 139.7)
+		(diameter 0)
+		(color 0 0 0 0)
+	)
+	(junction
+		(at 199.39 60.96)
+		(diameter 0)
+		(color 0 0 0 0)
+	)
+	(junction
+		(at 238.76 135.89)
+		(diameter 0)
+		(color 0 0 0 0)
+	)
+	(junction
+		(at 46.99 83.82)
+		(diameter 0)
+		(color 0 0 0 0)
+	)
+	(junction
+		(at 17.78 73.66)
+		(diameter 0)
+		(color 0 0 0 0)
+	)
+	(junction
+		(at 259.08 118.11)
+		(diameter 0)
+		(color 0 0 0 0)
+	)
+	(junction
+		(at 179.07 135.89)
+		(diameter 0)
+		(color 0 0 0 0)
+	)
+	(junction
+		(at 275.59 135.89)
+		(diameter 0)
+		(color 0 0 0 0)
+	)
+	(junction
+		(at 154.94 101.6)
+		(diameter 0)
+		(color 0 0 0 0)
+	)
+	(junction
+		(at 229.87 134.62)
+		(diameter 0)
+		(color 0 0 0 0)
+	)
+	(junction
+		(at 93.98 90.17)
+		(diameter 0)
+		(color 0 0 0 0)
+	)
+	(junction
+		(at 90.17 100.33)
+		(diameter 0)
+		(color 0 0 0 0)
+	)
+	(junction
+		(at 199.39 74.93)
+		(diameter 0)
+		(color 0 0 0 0)
+	)
+	(junction
+		(at 88.9 60.96)
+		(diameter 0)
+		(color 0 0 0 0)
+	)
+	(junction
+		(at 234.95 57.15)
+		(diameter 0)
+		(color 0 0 0 0)
+	)
+	(junction
+		(at 176.53 69.85)
+		(diameter 0)
+		(color 0 0 0 0)
 	)
 	(junction
@@
 	)
 	(junction
-		(at 19.05 71.12)
-		(diameter 0)
-		(color 0 0 0 0)
-	)
-	(junction
-		(at 154.94 109.22)
-		(diameter 0)
-		(color 0 0 0 0)
-	)
-	(junction
-		(at 15.24 88.9)
-		(diameter 0)
-		(color 0 0 0 0)
-	)
-	(junction
-		(at 245.11 118.11)
-		(diameter 0)
-		(color 0 0 0 0)
-	)
-	(junction
-		(at 139.7 144.78)
-		(diameter 0)
-		(color 0 0 0 0)
-	)
-	(junction
-		(at 196.85 95.25)
-		(diameter 0)
-		(color 0 0 0 0)
-	)
-	(junction
-		(at 148.59 82.55)
-		(diameter 0)
-		(color 0 0 0 0)
-	)
-	(junction
-		(at 151.13 109.22)
-		(diameter 0)
-		(color 0 0 0 0)
-	)
-	(junction
-		(at 189.23 115.57)
-		(diameter 0)
-		(color 0 0 0 0)
-	)
-	(junction
-		(at 232.41 82.55)
-		(diameter 0)
-		(color 0 0 0 0)
-	)
-	(junction
-		(at 154.94 92.71)
-		(diameter 0)
-		(color 0 0 0 0)
-	)
-	(junction
-		(at 110.49 83.82)
-		(diameter 0)
-		(color 0 0 0 0)
-	)
-	(junction
-		(at 152.4 53.34)
-		(diameter 0)
-		(color 0 0 0 0)
-	)
-	(junction
-		(at 181.61 139.7)
-		(diameter 0)
-		(color 0 0 0 0)
-	)
-	(junction
-		(at 199.39 60.96)
-		(diameter 0)
-		(color 0 0 0 0)
-	)
-	(junction
-		(at 238.76 135.89)
-		(diameter 0)
-		(color 0 0 0 0)
-	)
-	(junction
-		(at 46.99 83.82)
-		(diameter 0)
-		(color 0 0 0 0)
-	)
-	(junction
-		(at 17.78 73.66)
-		(diameter 0)
-		(color 0 0 0 0)
-	)
-	(junction
-		(at 259.08 118.11)
-		(diameter 0)
-		(color 0 0 0 0)
-	)
-	(junction
-		(at 179.07 135.89)
-		(diameter 0)
-		(color 0 0 0 0)
-	)
-	(junction
-		(at 275.59 135.89)
-		(diameter 0)
-		(color 0 0 0 0)
-	)
-	(junction
-		(at 154.94 101.6)
-		(diameter 0)
-		(color 0 0 0 0)
-	)
-	(junction
-		(at 229.87 134.62)
-		(diameter 0)
-		(color 0 0 0 0)
-	)
-	(junction
-		(at 93.98 90.17)
-		(diameter 0)
-		(color 0 0 0 0)
-	)
-	(junction
-		(at 90.17 100.33)
-		(diameter 0)
-		(color 0 0 0 0)
-	)
-	(junction
-		(at 199.39 74.93)
-		(diameter 0)
-		(color 0 0 0 0)
-	)
-	(junction
-		(at 88.9 60.96)
-		(diameter 0)
-		(color 0 0 0 0)
-	)
-	(junction
-		(at 234.95 57.15)
-		(diameter 0)
-		(color 0 0 0 0)
-	)
-	(junction
-		(at 176.53 69.85)
-		(diameter 0)
-		(color 0 0 0 0)
-	)
-	(junction
 		(at 138.43 121.92)
 		(diameter 0)
@@
 	(wire
 		(pts
-			(xy 157.48 60.96) (xy 166.37 60.96)
-		)
-		(stroke
-			(width 0)
-			(type default)
-		)
-	)
-	(wire
-		(pts
 			(xy 138.43 135.89) (xy 179.07 135.89)
 		)
@@
 	(wire
 		(pts
-			(xy 148.59 66.04) (xy 147.32 66.04)
-		)
-		(stroke
-			(width 0)
-			(type default)
-		)
-	)
-	(wire
-		(pts
 			(xy 247.65 129.54) (xy 238.76 129.54)
 		)
@@
 	(wire
 		(pts
+			(xy 148.59 66.04) (xy 157.48 66.04)
+		)
+		(stroke
+			(width 0)
+			(type default)
+		)
+	)
+	(wire
+		(pts
 			(xy 229.87 137.16) (xy 229.87 134.62)
 		)
@@
 	(wire
 		(pts
+			(xy 157.48 66.04) (xy 157.48 60.96)
+		)
+		(stroke
+			(width 0)
+			(type default)
+		)
+	)
+	(wire
+		(pts
 			(xy 16.51 76.2) (xy 16.51 96.52)
 		)
@@
 	(wire
 		(pts
+			(xy 166.37 55.88) (xy 166.37 60.96)
+		)
+		(stroke
+			(width 0)
+			(type default)
+		)
+	)
+	(wire
+		(pts
 			(xy 19.05 91.44) (xy 15.24 91.44)
 		)
@@
 	(wire
 		(pts
-			(xy 147.32 66.04) (xy 147.32 60.96)
-		)
-		(stroke
-			(width 0)
-			(type default)
-		)
-	)
-	(wire
-		(pts
 			(xy 176.53 60.96) (xy 176.53 58.42)
 		)
@@
 	(wire
 		(pts
+			(xy 147.32 60.96) (xy 147.32 55.88)
+		)
+		(stroke
+			(width 0)
+			(type default)
+		)
+	)
+	(wire
+		(pts
 			(xy 176.53 45.72) (xy 234.95 45.72)
 		)
@@
 		)
 		(stroke
+			(width 0)
+			(type default)
+		)
+	)
+	(wire
+		(pts
+			(xy 147.32 55.88) (xy 166.37 55.88)
+		)
+		(stroke
