File: FirstArdTest/Just theOLED/minithing/minithing.kicad_pcb (KiCad board)
At the start: 2 copper layers, 10 parts, among them Q1 NMOS, Q2 NMOS, Q3 FDN340P, U1 TP4056-42-ESOP8, U2 MT3608

Commit message: PCB Finish
Parts:
- removed D1: ESD441DPLR, SamacSys_Parts:ESD441DPLR
- added C1: 100uF, Capacitor_SMD:C_1206_3216Metric_Pad1.33x1.80mm_HandSolder, F.Cu at (60.0, 30.1)
- added C2: 0.1uF, Capacitor_SMD:C_0805_2012Metric_Pad1.18x1.45mm_HandSolder, F.Cu at (56.3, 30.6)
- added C3: 0.1uF, Capacitor_SMD:C_0805_2012Metric_Pad1.18x1.45mm_HandSolder, F.Cu at (87.9, 39.4)
- added C4: 22uF, Capacitor_SMD:C_1206_3216Metric_Pad1.33x1.80mm_HandSolder, F.Cu at (45.7, 28.6)
- added C5: 0.1uF, Capacitor_SMD:C_0805_2012Metric_Pad1.18x1.45mm_HandSolder, F.Cu at (70.8, 32.7)
- added C6: 0.1uF, Capacitor_SMD:C_0805_2012Metric_Pad1.18x1.45mm_HandSolder, F.Cu at (69.2, 39.4)
- added C7: 22uF, Capacitor_SMD:C_1206_3216Metric_Pad1.33x1.80mm_HandSolder, F.Cu at (77.9, 42.9)
- added C8: 0.1uF, Capacitor_SMD:C_0805_2012Metric_Pad1.18x1.45mm_HandSolder, F.Cu at (82.0, 43.4)
- added G***: LOGO, LOGO, F.Cu at (35.4, 47.2)
- added IC1: DS3231MZ+, SamacSys_Parts:SOIC127P600X175-8N, F.Cu at (96.7, 42.3)
- added J1: USB4110-GF-A, SamacSys_Parts:USB4110GFA, F.Cu at (29.8, 35.5)
- added L1: 4.7uH, Inductor_SMD:L_0805_2012Metric_Pad1.15x1.40mm_HandSolder, F.Cu at (74.1, 29.5)
- added LI-IONbatt1: BATTERY, Battery:BatteryHolder_Keystone_1042_1x18650, F.Cu at (67.5, 44.4)
- added R1: 5.1kR, Resistor_SMD:R_0805_2012Metric_Pad1.20x1.40mm_HandSolder, F.Cu at (42.9, 44.9)
- added R10: 1.2kR, Resistor_SMD:R_0805_2012Metric_Pad1.20x1.40mm_HandSolder, F.Cu at (56.6, 36.4)
- added R11: 1MR, Resistor_SMD:R_0805_2012Metric_Pad1.20x1.40mm_HandSolder, F.Cu at (70.8, 35.0)
- added R12: 1MR, Resistor_SMD:R_0805_2012Metric_Pad1.20x1.40mm_HandSolder, F.Cu at (71.6, 39.4)
- added R2: 5.1KR, Resistor_SMD:R_0805_2012Metric_Pad1.20x1.40mm_HandSolder, F.Cu at (40.2, 44.8)
- added R3: 100R, Resistor_SMD:R_0805_2012Metric_Pad1.20x1.40mm_HandSolder, F.Cu at (90.7, 41.6)
- added R4: 1k, Resistor_SMD:R_0805_2012Metric_Pad1.20x1.40mm_HandSolder, F.Cu at (87.9, 35.3)
- added R5: 110k, Resistor_SMD:R_0805_2012Metric_Pad1.20x1.40mm_HandSolder, F.Cu at (77.7, 38.4)
- added R6: 15k, Resistor_SMD:R_0805_2012Metric_Pad1.20x1.40mm_HandSolder, F.Cu at (75.0, 38.0)
- added R7: 1kR, Resistor_SMD:R_0805_2012Metric_Pad1.20x1.40mm_HandSolder, F.Cu at (57.9, 40.3)
- added R8: 1kR, Resistor_SMD:R_0805_2012Metric_Pad1.20x1.40mm_HandSolder, F.Cu at (67.8, 33.7)
- added R9: 0.4R, Resistor_SMD:R_1206_3216Metric_Pad1.30x1.75mm_HandSolder, F.Cu at (64.0, 30.1)
- added SW1: SW_Push, Button_Switch_THT:SW_PUSH_6mm, F.Cu at (30.8, 63.5)
- added SW2: SW_Push, Button_Switch_THT:SW_PUSH_6mm, F.Cu at (39.1, 63.5)
- added SW3: SW_Push, Button_Switch_THT:SW_PUSH_6mm_H4.3mm, F.Cu at (47.3, 63.5)
- added SW4: SW_Push, Button_Switch_THT:SW_PUSH_6mm, F.Cu at (55.5, 63.5)
- added U3: AHT20, SamacSys_Parts:AHT20, F.Cu at (48.5, 40.0)
- added U4: MCP23008-xSO, Package_SO:SOIC-18W_7.5x11.6mm_P1.27mm, F.Cu at (54.2, 49.1)
- added Z1: 1N4733A, SamacSys_Parts:DIOAD1405W86L465D235, F.Cu at (53.1, 41.5)
- D2, D3: footprint Diode_SMD:D_SMA -> Diode_SMD:D_SMC_Handsoldering
- U1: value TP4056-42-ESOP8 -> TP4056
- moved A1 42.0 mm to (66.8, 62.4), turned to 90 degrees
- moved Q3 39.0 mm to (69.7, 29.5)
- moved Q2 35.3 mm to (96.0, 29.9), turned to 180 degrees
- moved DW01A1 33.4 mm to (91.4, 34.9)
- moved Q1 29.4 mm to (90.2, 30.1)
- moved U1 24.4 mm to (62.2, 36.4)
- moved D2 16.9 mm to (39.5, 35.6)
- moved U2 16.2 mm to (76.3, 33.1), turned to 90 degrees
- moved D3 15.1 mm to (83.1, 34.5)
Connections:
- net Net-(D2-A2) renamed 1AMP
- net Net-(Q3-S) renamed BATTERY
- A1 pad 17: unconnected-(A1-3V3-Pad17) -> Net-(A1-3V3)
- A1 pad 23: unconnected-(A1-A4-Pad23) -> Net-(A1-A4)
- A1 pad 24: unconnected-(A1-A5-Pad24) -> Net-(A1-A5)
- A1 pad 29: CON.ARD -> GND
- A1 pad 4: CON.ARD -> GND
- A1 pad 5: CON.ARD -> GND
- A1 pad 6: CON.ARD -> Net-(A1-D3)
- D2 pad 1: CON.ARD -> GND
- DW01A1 pad 6: Net-(DW01A1-GND) -> GND
- Q1 pad 1: Net-(DW01A1-GND) -> GND
- Q1 pad 3: Net-(DW01A1-GND) -> GND
- Q2 pad 1: CON.ARD -> GND
- Q2 pad 3: CON.ARD -> GND
- U1 pad 1: CON.ARD -> GND
- U1 pad 3: CON.ARD -> GND
- U1 pad 6: CON.ARD -> GND
- U1 pad 7: CON.ARD -> Net-(A1-D3)
- U2 pad 2: CON.ARD -> GND
Routing:
- net BATTERY: track 0.00 -> 100.9 mm, vias 0 -> 2
- net Net-(A1-3V3): track 0.00 -> 72.5 mm
- net 1AMP: track 0.00 -> 65.2 mm, vias 0 -> 2
- net GND: track 0.00 -> 62.7 mm, vias 0 -> 12
- net Net-(A1-A5): track 0.00 -> 60.3 mm
- net Net-(A1-A4): track 0.00 -> 55.6 mm
- net Net-(A1-D4): track 0.00 -> 52.5 mm, vias 0 -> 1
- net Net-(A1-D3): track 0.00 -> 37.4 mm, vias 0 -> 1
- net Net-(U1-CE): track 0.00 -> 36.7 mm
- net Net-(U4-GP0): track 0.00 -> 26.1 mm
- net Net-(DW01A1-OC): track 0.00 -> 21.1 mm, vias 0 -> 2
- net Net-(U4-GP1): track 0.00 -> 19.7 mm
- net 5V out: track 0.00 -> 19.3 mm
- net Net-(J1-PadA5): track 0.00 -> 16.7 mm
- net Net-(DW01A1-OD): track 0.00 -> 16.4 mm
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- added copper zone on F.Cu, net GND
Other:
- board outline added: 81.8 x 40.2 mm
- board text added: "designed by candiedapple"
